Commit message: Refactored package layout

File: resources/robots/urdf/panda_arm.urdf (robot description, URDF)
Before this commit: robot panda, 10 links, 9 joints
Links:
- link panda_link0: geometry collision mesh filename=package://cfc_collision_app/resources/robots/meshes/panda/c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; visual mesh filename=package://cfc_collision_app/resources/robots/meshes/panda/v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
- link panda_link1: geometry collision mesh filename=package://cfc_collision_app/resources/robots/meshes/panda/c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; visual mesh filename=package://cfc_collision_app/resources/robots/meshes/panda/v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
- link panda_link2: geometry collision mesh filename=package://cfc_collision_app/resources/robots/meshes/panda/c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; visual mesh filename=package://cfc_collision_app/resources/robots/meshes/panda/v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
- link panda_link3: geometry collision mesh filename=package://cfc_collision_app/resources/robots/meshes/panda/c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; visual mesh filename=package://cfc_collision_app/resources/robots/meshes/panda/v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
- link panda_link4: geometry collision mesh filename=package://cfc_collision_app/resources/robots/meshes/panda/c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; visual mesh filename=package://cfc_collision_app/resources/robots/meshes/panda/v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
- link panda_link5: geometry collision mesh filename=package://cfc_collision_app/resources/robots/meshes/panda/c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; visual mesh filename=package://cfc_collision_app/resources/robots/meshes/panda/v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
- link panda_link6: geometry collision mesh filename=package://cfc_collision_app/resources/robots/meshes/panda/c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; visual mesh filename=package://cfc_collision_app/resources/robots/meshes/panda/v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
- link panda_link7: geometry collision mesh filename=package://cfc_collision_app/resources/robots/meshes/panda/c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; visual mesh filename=package://cfc_collision_app/resources/robots/meshes/panda/v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

File: resources/robots/urdf/panda_arm.xacro (robot description, xacro)
@@ -5,5 +5,5 @@
     <color rgba="1 1 1 1"/>
   </material>
-  <xacro:include filename="$(find cfc_collision_app)/resources/urdf/panda_arm_macro.xacro"/>
+  <xacro:include filename="$(find cfc_collision_app)/resources/robots/urdf/panda_arm_macro.xacro"/>
   <!-- box shaped table as base for Panda -->
   <link name="base">

File: resources/robots/urdf/panda_arm_macro.xacro (robot description, xacro)
@@ -4,4 +4,5 @@
   <!-- arm_id: Namespace of the panda arm. Serves to differentiate between arms in case of multiple instances. -->
   <xacro:macro name="panda_arm" params="arm_id:='panda' description_pkg:='cfc_collision_app' connected_to:='' xyz:='0 0 0' rpy:='0 0 0' safety_distance:=0">
+    <xacro:arg name='mesh_file_prefix' default="${description_pkg}/resources/robots/meshes/panda" />
     <xacro:unless value="${not connected_to}">
       <joint name="${arm_id}_joint_${connected_to}" type="fixed">
@@ -14,10 +15,10 @@
       <visual>
         <geometry>
-          <mesh filename="package://${description_pkg}/resources/meshes/panda/visual/link0.dae" />
+          <mesh filename="package://$(arg mesh_file_prefix)/visual/link0.dae" />
         </geometry>
         </visual>
       <collision>
         <geometry>
-          <mesh filename="package://${description_pkg}/resources/meshes/panda/collision/link0.stl" />
+          <mesh filename="package://$(arg mesh_file_prefix)/collision/link0.stl" />
         </geometry>
       </collision>
@@ -26,10 +27,10 @@
       <visual>
         <geometry>
-          <mesh filename="package://${description_pkg}/resources/meshes/panda/visual/link1.dae" />
+          <mesh filename="package://$(arg mesh_file_prefix)/visual/link1.dae" />
         </geometry>
       </visual>
       <collision>
         <geometry>
-          <mesh filename="package://${description_pkg}/resources/meshes/panda/collision/link1.stl" />
+          <mesh filename="package://$(arg mesh_file_prefix)/collision/link1.stl" />
         </geometry>
       </collision>
@@ -46,10 +47,10 @@
       <visual>
         <geometry>
-          <mesh filename="package://${description_pkg}/resources/meshes/panda/visual/link2.dae" />
+          <mesh filename="package://$(arg mesh_file_prefix)/visual/link2.dae" />
         </geometry>
       </visual>
       <collision>
         <geometry>
-          <mesh filename="package://${description_pkg}/resources/meshes/panda/collision/link2.stl" />
+          <mesh filename="package://$(arg mesh_file_prefix)/collision/link2.stl" />
         </geometry>
       </collision>
@@ -66,10 +67,10 @@
       <visual>
         <geometry>
-          <mesh filename="package://${description_pkg}/resources/meshes/panda/visual/link3.dae" />
+          <mesh filename="package://$(arg mesh_file_prefix)/visual/link3.dae" />
         </geometry>
       </visual>
       <collision>
         <geometry>
-          <mesh filename="package://${description_pkg}/resources/meshes/panda/collision/link3.stl" />
+          <mesh filename="package://$(arg mesh_file_prefix)/collision/link3.stl" />
         </geometry>
       </collision>
@@ -86,10 +87,10 @@
       <visual>
         <geometry>
-          <mesh filename="package://${description_pkg}/resources/meshes/panda/visual/link4.dae" />
+          <mesh filename="package://$(arg mesh_file_prefix)/visual/link4.dae" />
         </geometry>
       </visual>
       <collision>
         <geometry>
-          <mesh filename="package://${description_pkg}/resources/meshes/panda/collision/link4.stl" />
+          <mesh filename="package://$(arg mesh_file_prefix)/collision/link4.stl" />
         </geometry>
       </collision>
@@ -106,10 +107,10 @@
       <visual>
         <geometry>
-          <mesh filename="package://${description_pkg}/resources/meshes/panda/visual/link5.dae" />
+          <mesh filename="package://$(arg mesh_file_prefix)/visual/link5.dae" />
         </geometry>
       </visual>
       <collision>
         <geometry>
-          <mesh filename="package://${description_pkg}/resources/meshes/panda/collision/link5.stl" />
+          <mesh filename="package://$(arg mesh_file_prefix)/collision/link5.stl" />
         </geometry>
       </collision>
@@ -126,10 +127,10 @@
       <visual>
         <geometry>
-          <mesh filename="package://${description_pkg}/resources/meshes/panda/visual/link6.dae" />
+          <mesh filename="package://$(arg mesh_file_prefix)/visual/link6.dae" />
         </geometry>
       </visual>
       <collision>
         <geometry>
-          <mesh filename="package://${description_pkg}/resources/meshes/panda/collision/link6.stl" />
+          <mesh filename="package://$(arg mesh_file_prefix)/collision/link6.stl" />
         </geometry>
       </collision>
@@ -146,10 +147,10 @@
       <visual>
         <geometry>
-          <mesh filename="package://${description_pkg}/resources/meshes/panda/visual/link7.dae" />
+          <mesh filename="package://$(arg mesh_file_prefix)/visual/link7.dae" />
         </geometry>
       </visual>
       <collision>
         <geometry>
-          <mesh filename="package://${description_pkg}/resources/meshes/panda/collision/link7.stl" />
+          <mesh filename="package://$(arg mesh_file_prefix)/collision/link7.stl" />
         </geometry>
       </collision>

File: resources/robots/urdf/panda_dual_arm.urdf (robot description, URDF)
Before this commit: robot panda, 19 links, 18 joints
Links:
- link panda_1_link0: geometry collision mesh filename=package://cfc_collision_app/resources/robots/meshes/panda/c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; visual mesh filename=package://cfc_collision_app/resources/robots/meshes/panda/v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
- link panda_1_link1: geometry collision mesh filename=package://cfc_collision_app/resources/robots/meshes/panda/c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; visual mesh filename=package://cfc_collision_app/resources/robots/meshes/panda/v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
- link panda_1_link2: geometry collision mesh filename=package://cfc_collision_app/resources/robots/meshes/panda/c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; visual mesh filename=package://cfc_collision_app/resources/robots/meshes/panda/v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
- link panda_1_link3: geometry collision mesh filename=package://cfc_collision_app/resources/robots/meshes/panda/c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; visual mesh filename=package://cfc_collision_app/resources/robots/meshes/panda/v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
- link panda_1_link4: geometry collision mesh filename=package://cfc_collision_app/resources/robots/meshes/panda/c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; visual mesh filename=package://cfc_collision_app/resources/robots/meshes/panda/v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
- link panda_1_link5: geometry collision mesh filename=package://cfc_collision_app/resources/robots/meshes/panda/c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; visual mesh filename=package://cfc_collision_app/resources/robots/meshes/panda/v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
- link panda_1_link6: geometry collision mesh filename=package://cfc_collision_app/resources/robots/meshes/panda/c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; visual mesh filename=package://cfc_collision_app/resources/robots/meshes/panda/v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
- link panda_1_link7: geometry collision mesh filename=package://cfc_collision_app/resources/robots/meshes/panda/c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; visual mesh filename=package://cfc_collision_app/resources/robots/meshes/panda/v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
- link panda_2_link0: geometry collision mesh filename=package://cfc_collision_app/resources/robots/meshes/panda/c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; visual mesh filename=package://cfc_collision_app/resources/robots/meshes/panda/v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
- link panda_2_link1: geometry collision mesh filename=package://cfc_collision_app/resources/robots/meshes/panda/c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; visual mesh filename=package://cfc_collision_app/resources/robots/meshes/panda/v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
- link panda_2_link2: geometry collision mesh filename=package://cfc_collision_app/resources/robots/meshes/panda/c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; visual mesh filename=package://cfc_collision_app/resources/robots/meshes/panda/v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
- link panda_2_link3: geometry collision mesh filename=package://cfc_collision_app/resources/robots/meshes/panda/c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; visual mesh filename=package://cfc_collision_app/resources/robots/meshes/panda/v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
- link panda_2_link4: geometry collision mesh filename=package://cfc_collision_app/resources/robots/meshes/panda/c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; visual mesh filename=package://cfc_collision_app/resources/robots/meshes/panda/v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
- link panda_2_link5: geometry collision mesh filename=package://cfc_collision_app/resources/robots/meshes/panda/c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; visual mesh filename=package://cfc_collision_app/resources/robots/meshes/panda/v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
- link panda_2_link6: geometry collision mesh filename=package://cfc_collision_app/resources/robots/meshes/panda/c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; visual mesh filename=package://cfc_collision_app/resources/robots/meshes/panda/v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
- link panda_2_link7: geometry collision mesh filename=package://cfc_collision_app/resources/robots/meshes/panda/c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; visual mesh filename=package://cfc_collision_app/resources/robots/meshes/panda/v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

File: resources/robots/urdf/panda_dual_arm.xacro (robot description, xacro)
@@ -3,5 +3,5 @@
   <xacro:arg name="arm_id_1" default="panda_1" />
   <xacro:arg name="arm_id_2" default="panda_2" />
-  <xacro:include filename="$(find cfc_collision_app)/resources/urdf/panda_arm_macro.xacro"/>
+  <xacro:include filename="$(find cfc_collision_app)/resources/robots/urdf/panda_arm_macro.xacro"/>
   <!-- box shaped table as base for the 2 Pandas -->
   <link name="base">

Commit message: Renamed package

File: resources/robots/urdf/panda_arm.urdf (robot description, URDF)
Before this commit: robot panda, 10 links, 9 joints
Links:
- link panda_link0: geometry collision mesh filename=package://cfc_collision_ros/resources/robots/meshes/panda/c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; visual mesh filename=package://cfc_collision_ros/resources/robots/meshes/panda/v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
- link panda_link1: geometry collision mesh filename=package://cfc_collision_ros/resources/robots/meshes/panda/c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; visual mesh filename=package://cfc_collision_ros/resources/robots/meshes/panda/v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
- link panda_link2: geometry collision mesh filename=package://cfc_collision_ros/resources/robots/meshes/panda/c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; visual mesh filename=package://cfc_collision_ros/resources/robots/meshes/panda/v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
- link panda_link3: geometry collision mesh filename=package://cfc_collision_ros/resources/robots/meshes/panda/c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; visual mesh filename=package://cfc_collision_ros/resources/robots/meshes/panda/v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
- link panda_link4: geometry collision mesh filename=package://cfc_collision_ros/resources/robots/meshes/panda/c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; visual mesh filename=package://cfc_collision_ros/resources/robots/meshes/panda/v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
- link panda_link5: geometry collision mesh filename=package://cfc_collision_ros/resources/robots/meshes/panda/c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; visual mesh filename=package://cfc_collision_ros/resources/robots/meshes/panda/v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
- link panda_link6: geometry collision mesh filename=package://cfc_collision_ros/resources/robots/meshes/panda/c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; visual mesh filename=package://cfc_collision_ros/resources/robots/meshes/panda/v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
- link panda_link7: geometry collision mesh filename=package://cfc_collision_ros/resources/robots/meshes/panda/c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; visual mesh filename=package://cfc_collision_ros/resources/robots/meshes/panda/v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

File: resources/robots/urdf/panda_arm.xacro (robot description, xacro)
@@ -5,5 +5,5 @@
     <color rgba="1 1 1 1"/>
   </material>
-  <xacro:include filename="$(find cfc_collision_app)/resources/robots/urdf/panda_arm_macro.xacro"/>
+  <xacro:include filename="$(find cfc_collision_ros)/resources/robots/urdf/panda_arm_macro.xacro"/>
   <!-- box shaped table as base for Panda -->
   <link name="base">

File: resources/robots/urdf/panda_arm_macro.xacro (robot description, xacro)
@@ -3,5 +3,5 @@
   <!-- safety_distance: Minimum safety distance in [m] by which the collision volumes are expanded and which is enforced during robot motions -->
   <!-- arm_id: Namespace of the panda arm. Serves to differentiate between arms in case of multiple instances. -->
-  <xacro:macro name="panda_arm" params="arm_id:='panda' description_pkg:='cfc_collision_app' connected_to:='' xyz:='0 0 0' rpy:='0 0 0' safety_distance:=0">
+  <xacro:macro name="panda_arm" params="arm_id:='panda' description_pkg:='cfc_collision_ros' connected_to:='' xyz:='0 0 0' rpy:='0 0 0' safety_distance:=0">
     <xacro:arg name='mesh_file_prefix' default="${description_pkg}/resources/robots/meshes/panda" />
     <xacro:unless value="${not connected_to}">

File: resources/robots/urdf/panda_dual_arm.urdf (robot description, URDF)
Before this commit: robot panda, 19 links, 18 joints
Links:
- link panda_1_link0: geometry collision mesh filename=package://cfc_collision_ros/resources/robots/meshes/panda/c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; visual mesh filename=package://cfc_collision_ros/resources/robots/meshes/panda/v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
- link panda_1_link1: geometry collision mesh filename=package://cfc_collision_ros/resources/robots/meshes/panda/c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; visual mesh filename=package://cfc_collision_ros/resources/robots/meshes/panda/v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
- link panda_1_link2: geometry collision mesh filename=package://cfc_collision_ros/resources/robots/meshes/panda/c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; visual mesh filename=package://cfc_collision_ros/resources/robots/meshes/panda/v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
- link panda_1_link3: geometry collision mesh filename=package://cfc_collision_ros/resources/robots/meshes/panda/c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; visual mesh filename=package://cfc_collision_ros/resources/robots/meshes/panda/v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
- link panda_1_link4: geometry collision mesh filename=package://cfc_collision_ros/resources/robots/meshes/panda/c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; visual mesh filename=package://cfc_collision_ros/resources/robots/meshes/panda/v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
- link panda_1_link5: geometry collision mesh filename=package://cfc_collision_ros/resources/robots/meshes/panda/c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; visual mesh filename=package://cfc_collision_ros/resources/robots/meshes/panda/v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
- link panda_1_link6: geometry collision mesh filename=package://cfc_collision_ros/resources/robots/meshes/panda/c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; visual mesh filename=package://cfc_collision_ros/resources/robots/meshes/panda/v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
- link panda_1_link7: geometry collision mesh filename=package://cfc_collision_ros/resources/robots/meshes/panda/c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; visual mesh filename=package://cfc_collision_ros/resources/robots/meshes/panda/v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
- link panda_2_link0: geometry collision mesh filename=package://cfc_collision_ros/resources/robots/meshes/panda/c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; visual mesh filename=package://cfc_collision_ros/resources/robots/meshes/panda/v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
- link panda_2_link1: geometry collision mesh filename=package://cfc_collision_ros/resources/robots/meshes/panda/c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; visual mesh filename=package://cfc_collision_ros/resources/robots/meshes/panda/v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
- link panda_2_link2: geometry collision mesh filename=package://cfc_collision_ros/resources/robots/meshes/panda/c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; visual mesh filename=package://cfc_collision_ros/resources/robots/meshes/panda/v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
- link panda_2_link3: geometry collision mesh filename=package://cfc_collision_ros/resources/robots/meshes/panda/c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; visual mesh filename=package://cfc_collision_ros/resources/robots/meshes/panda/v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
- link panda_2_link4: geometry collision mesh filename=package://cfc_collision_ros/resources/robots/meshes/panda/c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; visual mesh filename=package://cfc_collision_ros/resources/robots/meshes/panda/v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
- link panda_2_link5: geometry collision mesh filename=package://cfc_collision_ros/resources/robots/meshes/panda/c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; visual mesh filename=package://cfc_collision_ros/resources/robots/meshes/panda/v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
- link panda_2_link6: geometry collision mesh filename=package://cfc_collision_ros/resources/robots/meshes/panda/c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; visual mesh filename=package://cfc_collision_ros/resources/robots/meshes/panda/v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
- link panda_2_link7: geometry collision mesh filename=package://cfc_collision_ros/resources/robots/meshes/panda/c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; visual mesh filename=package://cfc_collision_ros/resources/robots/meshes/panda/v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

File: resources/robots/urdf/panda_dual_arm.xacro (robot description, xacro)
@@ -3,5 +3,5 @@
   <xacro:arg name="arm_id_1" default="panda_1" />
   <xacro:arg name="arm_id_2" default="panda_2" />
-  <xacro:include filename="$(find cfc_collision_app)/resources/robots/urdf/panda_arm_macro.xacro"/>
+  <xacro:include filename="$(find cfc_collision_ros)/resources/robots/urdf/panda_arm_macro.xacro"/>
   <!-- box shaped table as base for the 2 Pandas -->
   <link name="base">
